Commit message: Part N

File: body.urdf (robot description, URDF)
Before this commit: robot robot, 3 links, 2 joints
Links:
- added link LBL, mass 1; collision box size=0.2 0.2 1; visual box size=0.2 0.2 1
- added link LFL, mass 1; collision box size=0.2 0.2 1; visual box size=0.2 0.2 1
- added link LLL, mass 1; collision box size=0.2 0.2 1; visual box size=0.2 0.2 1
- added link LRL, mass 1; collision box size=0.2 0.2 1; visual box size=0.2 0.2 1
- added link LeftLeg, mass 1; collision box size=1 0.2 0.2; visual box size=1 0.2 0.2
- added link RightLeg, mass 1; collision box size=1 0.2 0.2; visual box size=1 0.2 0.2
- link BackLeg: geometry collision box size=0.2 1 0.2; visual box size=0.2 1 0.2
- link FrontLeg: geometry collision box size=0.2 1 0.2; visual box size=0.2 1 0.2
Joints:
- added joint BackLeg_LBL: type revolute, parent BackLeg, child LBL, origin xyz=0 -1 0 rpy=0 0 0, axis 1 0 0, limit lower=-3.14159 upper=3.14159 effort=0.0 velocity=0.0
- added joint FrontLeg_LFL: type revolute, parent FrontLeg, child LFL, origin xyz=0 1 0 rpy=0 0 0, axis 1 0 0, limit lower=-3.14159 upper=3.14159 effort=0.0 velocity=0.0
- added joint LeftLeg_LLL: type revolute, parent LeftLeg, child LLL, origin xyz=-1 0 0 rpy=0 0 0, axis 0 1 0, limit lower=-3.14159 upper=3.14159 effort=0.0 velocity=0.0
- added joint RightLeg_LRL: type revolute, parent RightLeg, child LRL, origin xyz=1 0 0 rpy=0 0 0, axis 0, 1 0, limit lower=-3.14159 upper=3.14159 effort=0.0 velocity=0.0
- added joint Torso_LeftLeg: type revolute, parent Torso, child LeftLeg, origin xyz=-0.5 0 1 rpy=0 0 0, axis 0 1 0, limit lower=-3.14159 upper=3.14159 effort=0.0 velocity=0.0
- added joint Torso_RightLeg: type revolute, parent Torso, child RightLeg, origin xyz=0.5 0 1 rpy=0 0 0, axis 0 1 0, limit lower=-3.14159 upper=3.14159 effort=0.0 velocity=0.0
- joint Torso_BackLeg: axis 0 1 0 -> 1 0 0; origin xyz=1 0 1 rpy=0 0 0 -> xyz=0 -0.5 1 rpy=0 0 0
- joint Torso_FrontLeg: axis 0 1 0 -> 1 0 0; origin xyz=2 0 1 rpy=0 0 0 -> xyz=0 0.5 1 rpy=0 0 0

Commit message: Assignment 5

File: body.urdf (robot description, URDF)
Before this commit: robot robot, 9 links, 8 joints
Links:
- removed link BackLeg
- removed link FrontLeg
- removed link LBL
- removed link LFL
- removed link LLL
- removed link LRL
- removed link LeftLeg
- removed link RightLeg
- removed link Torso
- added link A, mass 1; collision box size=1 1 1; visual box size=1 1 1
- added link B1, mass 1; collision box size=0.2 1 0.2; visual box size=0.2 1 0.2
- added link B2, mass 1; collision box size=0.2 0.2 1; visual box size=0.2 0.2 1
- added link C1, mass 1; collision box size=0.2 1 0.2; visual box size=0.2 1 0.2
- added link C2, mass 1; collision box size=0.2 0.2 1; visual box size=0.2 0.2 1
- added link D, mass 1; collision box size=0.2 0.2 0.5; visual box size=0.2 0.2 0.5
Joints:
- removed joint BackLeg_LBL
- removed joint FrontLeg_LFL
- removed joint LeftLeg_LLL
- removed joint RightLeg_LRL
- removed joint Torso_BackLeg
- removed joint Torso_FrontLeg
- removed joint Torso_LeftLeg
- removed joint Torso_RightLeg
- added joint A_B1: type revolute, parent A, child B1, origin xyz=0 -0.5 1 rpy=0 0 0, axis 0 1 0, limit lower=-3.14159 upper=3.14159 effort=0.0 velocity=0.0
- added joint A_C1: type revolute, parent A, child C1, origin xyz=0 0.5 1 rpy=0 0 0, axis 0 1 0, limit lower=-3.14159 upper=3.14159 effort=0.0 velocity=0.0
- added joint A_D: type revolute, parent A, child D, origin xyz=0 0 0.5 rpy=0 0 0, axis 0 1 0, limit lower=-3.14159 upper=3.14159 effort=0.0 velocity=0.0
- added joint B1_B2: type revolute, parent B1, child B2, origin xyz=0 -1 0 rpy=0 0 0, axis 1 0 0, limit lower=-3.14159 upper=3.14159 effort=0.0 velocity=0.0
- added joint C1_C2: type revolute, parent C1, child C2, origin xyz=0 1 0 rpy=0 0 0, axis 1 0 0, limit lower=-3.14159 upper=3.14159 effort=0.0 velocity=0.0
