Commit message: Training finished
Trained 10 new seeds. Bodies start out smaller, 10 pop x 500 gens.
Fixed a bug where the brain was mutated even though it was empty.
Updated demo to allow the user to specify which seed is played back.

File: body_evolved_1.urdf (robot description, URDF)
Before this commit: robot robot, 10 links, 9 joints
Links:
- removed link 11
- removed link 12
- added link 6, mass 1; collision box size=0.6074635117277701 0.8902115543282348 0.9743433912068795; visual box size=0.6074635117277701 0.8902115543282348 0.9743433912068795
- link 0: geometry collision box size=0.7435969545367118 0.7099967760051205 0.6309998523596678; visual box size=0.7435969545367118 0.7099967760051205 0.6309998523596678
- link 1: geometry collision box size=0.6017169121850453 0.9481612784020024 0.9365471891348203; visual box size=0.6017169121850453 0.9481612784020024 0.9365471891348203
- link 2: geometry collision box size=0.5590963146735193 0.9184988911067561 0.8720679606847677; visual box size=0.5590963146735193 0.9184988911067561 0.8720679606847677
- link 3: geometry collision box size=0.6910503212745698 0.5633566919234614 0.6221333316044879; visual box size=0.6910503212745698 0.5633566919234614 0.6221333316044879
- link 4: geometry collision box size=0.9433730061865055 0.5972556425614559 0.7149025258849349; visual box size=0.9433730061865055 0.5972556425614559 0.7149025258849349
- link 5: geometry collision box size=0.8022816282990718 0.7755659618118593 0.8750765721289209; visual box size=0.8022816282990718 0.7755659618118593 0.8750765721289209
- link 7: geometry collision box size=0.9674550718908375 0.7348431421006203 0.8985943033378424; visual box size=0.9674550718908375 0.7348431421006203 0.8985943033378424
- link root: geometry collision box size=0.996350436832409 0.7594021253667071 0.5861398507385627; visual box size=0.996350436832409 0.7594021253667071 0.5861398507385627
Joints:
- removed joint 0_2
- removed joint 1_5
- removed joint 2_3
- removed joint 3_12
- removed joint 4_11
- removed joint root_4
- removed joint root_7
- added joint 2_4: type revolute, parent 2, child 4, origin xyz=0.0 0.9184988911067561 0.0 rpy=0 0 0, axis 0 1 0, limit lower=-3.14159 upper=3.14159 effort=0.0 velocity=0.0
- added joint 4_5: type revolute, parent 4, child 5, origin xyz=-0.4716865030932528 0.29862782128072796 0.0 rpy=0 0 0, axis 1 0 0, limit lower=-3.14159 upper=3.14159 effort=0.0 velocity=0.0
- added joint 5_6: type revolute, parent 5, child 6, origin xyz=-0.8022816282990718 0.0 0.0 rpy=0 0 0, axis 1 0 0, limit lower=-3.14159 upper=3.14159 effort=0.0 velocity=0.0
- added joint 6_7: type revolute, parent 6, child 7, origin xyz=-0.6074635117277701 0.0 0.0 rpy=0 0 0, axis 0 0 1, limit lower=-3.14159 upper=3.14159 effort=0.0 velocity=0.0
- added joint root_2: type revolute, parent root, child 2, origin xyz=0.0 0.3797010626833536 2.0 rpy=0 0 0, axis 1 0 0, limit lower=-3.14159 upper=3.14159 effort=0.0 velocity=0.0
- added joint root_3: type revolute, parent root, child 3, origin xyz=0.0 0.0 2.2930699253692812 rpy=0 0 0, axis 0 1 0, limit lower=-3.14159 upper=3.14159 effort=0.0 velocity=0.0
- joint root_0: axis 1 0 0 -> 0 1 0; origin xyz=0.4961449447401765 0.0 2.0 rpy=0 0 0 -> xyz=0.0 0.0 1.7069300746307188 rpy=0 0 0
- joint root_1: origin xyz=0.0 -0.29735450551093845 2.0 rpy=0 0 0 -> xyz=0.4981752184162045 0.0 2.0 rpy=0 0 0

File: body_evolved_2.urdf (robot description, URDF)
Before this commit: robot robot, 14 links, 13 joints
Links:
- removed link 11
- removed link 12
- removed link 13
- removed link 4
- removed link 6
- removed link 8
- removed link 9
- link 0: geometry collision box size=0.5290080401814274 0.6578403807744916 0.7927631668339294; visual box size=0.5290080401814274 0.6578403807744916 0.7927631668339294
- link 1: geometry collision box size=0.5748113694184736 0.519870400673137 0.5990067440868715; visual box size=0.5748113694184736 0.519870400673137 0.5990067440868715
- link 2: geometry collision box size=0.594890153101143 0.5590280982655821 0.812770690855237; visual box size=0.594890153101143 0.5590280982655821 0.812770690855237
- link 3: geometry collision box size=0.5135854638936521 0.6496043578604149 0.8918507072632531; visual box size=0.5135854638936521 0.6496043578604149 0.8918507072632531
- link 5: geometry collision box size=0.5261412214483974 0.5872079022360928 0.6312474591073177; visual box size=0.5261412214483974 0.5872079022360928 0.6312474591073177
- link 7: geometry collision box size=0.8053416158708253 0.5568430304914274 0.9352451906453798; visual box size=0.8053416158708253 0.5568430304914274 0.9352451906453798
- link root: geometry collision box size=0.9447909556142241 0.886285692090284 0.7647709888482697; visual box size=0.9447909556142241 0.886285692090284 0.7647709888482697
Joints:
- removed joint 0_1
- removed joint 0_7
- removed joint 1_4
- removed joint 2_5
- removed joint 2_6
- removed joint 5_9
- removed joint 6_8
- removed joint 8_11
- removed joint 8_13
- removed joint 9_12
- removed joint root_3
- added joint 0_5: type revolute, parent 0, child 5, origin xyz=0.2645040200907137 -0.3289201903872458 0.0 rpy=0 0 0, axis 0 0 1, limit lower=-3.14159 upper=3.14159 effort=0.0 velocity=0.0
- added joint 2_3: type revolute, parent 2, child 3, origin xyz=-0.2974450765505715 -0.27951404913279104 0.0 rpy=0 0 0, axis 1 0 0, limit lower=-3.14159 upper=3.14159 effort=0.0 velocity=0.0
- added joint 2_7: type revolute, parent 2, child 7, origin xyz=-0.594890153101143 0.0 0.0 rpy=0 0 0, axis 0 0 1, limit lower=-3.14159 upper=3.14159 effort=0.0 velocity=0.0
- added joint root_1: type revolute, parent root, child 1, origin xyz=0.0 0.0 1.6176145055758653 rpy=0 0 0, axis 0 0 1, limit lower=-3.14159 upper=3.14159 effort=0.0 velocity=0.0
- joint root_0: axis 1 0 0 -> 0 1 0; origin xyz=0.2798382605098541 0.0 2.0 rpy=0 0 0 -> xyz=0.47239547780711205 0.0 2.0 rpy=0 0 0
- joint root_2: axis 0 1 0 -> 0 0 1; origin xyz=-0.2798382605098541 0.0 2.0 rpy=0 0 0 -> xyz=-0.47239547780711205 0.0 2.0 rpy=0 0 0

File: body_evolved_3.urdf (robot description, URDF)
Before this commit: robot robot, 7 links, 6 joints
Links:
- removed link 2
- removed link 6
- removed link 9
- added link 4, mass 1; collision box size=0.789948181979392 0.8089617990561951 0.6353355574300554; visual box size=0.789948181979392 0.8089617990561951 0.6353355574300554
- link 0: geometry collision box size=0.9964027271981054 0.9628027407039228 0.8374351913517831; visual box size=0.9964027271981054 0.9628027407039228 0.8374351913517831
- link 1: geometry collision box size=0.800938624422185 0.8912577213701942 0.7746632906599691; visual box size=0.800938624422185 0.8912577213701942 0.7746632906599691
- link 3: geometry collision box size=0.6850907888847471 0.7851949086025148 0.7096083993455649; visual box size=0.6850907888847471 0.7851949086025148 0.7096083993455649
- link root: geometry collision box size=0.7634271049907806 0.6173534887046259 0.9342220466702944; visual box size=0.7634271049907806 0.6173534887046259 0.9342220466702944
Joints:
- removed joint 1_2
- removed joint 2_3
- removed joint 2_9
- removed joint 3_6
- added joint 0_3: type revolute, parent 0, child 3, origin xyz=-0.4982013635990527 0.4814013703519614 0.0 rpy=0 0 0, axis 0 1 0, limit lower=-3.14159 upper=3.14159 effort=0.0 velocity=0.0
- added joint 3_4: type revolute, parent 3, child 4, origin xyz=0.0 0.7851949086025148 0.0 rpy=0 0 0, axis 0 1 0, limit lower=-3.14159 upper=3.14159 effort=0.0 velocity=0.0
- joint 0_1: axis 1 0 0 -> 0 1 0; origin xyz=0.0 0.0 0.7903012277930048 rpy=0 0 0 -> xyz=-0.4982013635990527 0.0 -0.41871759567589156 rpy=0 0 0
- joint root_0: axis 0 1 0 -> 0 0 1; origin xyz=0.0 0.0 2.461776489419796 rpy=0 0 0 -> xyz=-0.3817135524953903 0.0 2.0 rpy=0 0 0

File: body_evolved_4.urdf (robot description, URDF)
Before this commit: robot robot, 13 links, 12 joints
Links:
- removed link 12
- removed link 13
- removed link 14
- removed link 3
- removed link 6
- removed link 8
- removed link 9
- link 0: geometry collision box size=0.6482045105476706 0.6694653574255502 0.6474795002330811; visual box size=0.6482045105476706 0.6694653574255502 0.6474795002330811
- link 1: geometry collision box size=0.9115104635451853 0.9153476039226043 0.5537964581797001; visual box size=0.9115104635451853 0.9153476039226043 0.5537964581797001
- link 2: geometry collision box size=0.7029807259785211 0.7963582992683782 0.8261248961658333; visual box size=0.7029807259785211 0.7963582992683782 0.8261248961658333
- link 4: geometry collision box size=0.6047645029343117 0.6021533893767133 0.5411518444727321; visual box size=0.6047645029343117 0.6021533893767133 0.5411518444727321
- link 5: geometry collision box size=0.8292926386140498 0.8158589914709867 0.952296386668839; visual box size=0.8292926386140498 0.8158589914709867 0.952296386668839
- link root: geometry collision box size=0.9525889626595079 0.9128809533429603 0.627328542582006; visual box size=0.9525889626595079 0.9128809533429603 0.627328542582006
Joints:
- removed joint 0_1
- removed joint 1_12
- removed joint 1_2
- removed joint 1_3
- removed joint 2_4
- removed joint 2_6
- removed joint 4_5
- removed joint 4_9
- removed joint 5_8
- removed joint 8_14
- removed joint root_13
- added joint 1_4: type revolute, parent 1, child 4, origin xyz=-0.45575523177259264 0.0 -0.27689822908985007 rpy=0 0 0, axis 0 1 0, limit lower=-3.14159 upper=3.14159 effort=0.0 velocity=0.0
- added joint 1_5: type revolute, parent 1, child 5, origin xyz=-0.45575523177259264 0.45767380196130214 0.0 rpy=0 0 0, axis 0 0 1, limit lower=-3.14159 upper=3.14159 effort=0.0 velocity=0.0
- added joint root_1: type revolute, parent root, child 1, origin xyz=-0.47629448132975394 0.0 2.0 rpy=0 0 0, axis 0 1 0, limit lower=-3.14159 upper=3.14159 effort=0.0 velocity=0.0
- added joint root_2: type revolute, parent root, child 2, origin xyz=0.47629448132975394 0.0 2.0 rpy=0 0 0, axis 0 1 0, limit lower=-3.14159 upper=3.14159 effort=0.0 velocity=0.0
- joint root_0: axis 0 0 1 -> 1 0 0; origin xyz=0.0 -0.4024825587442714 2.0 rpy=0 0 0 -> xyz=0.0 0.0 1.686335728708997 rpy=0 0 0

File: body_evolved_5.urdf (robot description, URDF)
Before this commit: robot robot, 10 links, 9 joints
Links:
- removed link 10
- removed link 11
- removed link 12
- removed link 3
- removed link 4
- removed link 8
- removed link 9
- link 0: geometry collision box size=0.6232802723628615 0.7230923717572199 0.6725986237414099; visual box size=0.6232802723628615 0.7230923717572199 0.6725986237414099
- link 5: geometry collision box size=0.5262400149339639 0.8081715781397052 0.6897669217202689; visual box size=0.5262400149339639 0.8081715781397052 0.6897669217202689
- link root: geometry collision box size=0.7376134435339179 0.5571665267309669 0.8743253002344753; visual box size=0.7376134435339179 0.5571665267309669 0.8743253002344753
Joints:
- removed joint 11_12
- removed joint 3_4
- removed joint 3_9
- removed joint 4_5
- removed joint 4_8
- removed joint 5_11
- removed joint 8_10
- removed joint root_3
- added joint 0_5: type revolute, parent 0, child 5, origin xyz=-0.31164013618143077 0.0 -0.33629931187070494 rpy=0 0 0, axis 0 1 0, limit lower=-3.14159 upper=3.14159 effort=0.0 velocity=0.0
- joint root_0: axis 0 0 1 -> 0 1 0; origin xyz=-0.4979290501886772 0.0 2.0 rpy=0 0 0 -> xyz=-0.36880672176695894 0.0 2.0 rpy=0 0 0
